File: circuit/multiplex_driver.sch (KiCad schematic (older format))
At the start: 39 parts, among them IC1 ATTINY84-S, P1 ISCP, P2 I2C, P4 Anodes, P5 Cathod 1-8, P6 Cathode 9-16, P7 Serial, Q1 BC546A, Q2 BC546A, SW1 RESET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

Commit message: Added input for keypad
the uno model includes the ability to connect to a keypad.
Parts:
- removed IC1: ATTINY84-S, SO-14, symbol ATTINY84-S
- removed P1: ISCP, ~, symbol ISCP
- removed U?: 74HC595-16-PIN, ~, symbol 74HC595-16-PIN
- added P1: Keypad, symbol CONN_8
- added P3: +5V, symbol CONN_2
- added R11, R12, R13, R14, R15, R16, R17, R18: 10K, ~, symbol R
- added U9: CD4021B, ~, symbol CD4021B
- P5: value Cathod 1-8 -> Cathode 1-8
- P8: renamed from P?; value CONN_2 -> +24V
Connections:
- net labels added: K-RCLK, K-SER, K-SRCLK, M-ON/OFF, M-RCLK, M-SENSE, M-SER, M-SRCLK
- net labels removed: ON/OFF, SENSE
- wire segments 252 -> 263
- no-connect marks 3 -> 19
Other:
- moved on the sheet: C1, C2, D1, P2, P4, P5, P6, P7, P8, R1, R2, SHIELD1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

Commit message: Added pins for pr28v
Parts:
- added P?: pr28v, symbol CONN_4
Changed lines of the file:
@@
 Sheet 1 1
 Title ""
-Date "23 jan 2015"
+Date "25 jan 2015"
 Rev ""
 Comp ""
@@
 	1550 1600 1950 1600
 Connection ~ 1950 1600
+$Comp
+L CONN_4 P?
+U 1 1 54C4FA0B
+P 7650 6750
+F 0 "P?" V 7600 6750 50  0000 C CNN
+F 1 "pr28v" V 7700 6750 50  0000 C CNN
+F 2 "" H 7650 6750 60  0000 C CNN
+F 3 "" H 7650 6750 60  0000 C CNN
+	1    7650 6750
+	1    0    0    -1
+$EndComp
+$Comp
+L +5V #PWR?
+U 1 1 54C4FA18
+P 7300 6600
+F 0 "#PWR?" H 7300 6690 20  0001 C CNN
+F 1 "+5V" H 7300 6690 30  0000 C CNN
+F 2 "" H 7300 6600 60  0000 C CNN
+F 3 "" H 7300 6600 60  0000 C CNN
+	1    7300 6600
+	0    -1   -1   0
+$EndComp
+$Comp
+L GND #PWR?
+U 1 1 54C4FA1E
+P 7300 6900
+F 0 "#PWR?" H 7300 6900 30  0001 C CNN
+F 1 "GND" H 7300 6830 30  0001 C CNN
+F 2 "" H 7300 6900 60  0000 C CNN
+F 3 "" H 7300 6900 60  0000 C CNN
+	1    7300 6900
+	0    1    1    0
+$EndComp
+$Comp
+L GND #PWR?
+U 1 1 54C4FA24
+P 7300 6800
+F 0 "#PWR?" H 7300 6800 30  0001 C CNN
+F 1 "GND" H 7300 6730 30  0001 C CNN
+F 2 "" H 7300 6800 60  0000 C CNN
+F 3 "" H 7300 6800 60  0000 C CNN
+	1    7300 6800
+	0    1    1    0
+$EndComp
+$Comp
+L +24V #PWR?
+U 1 1 54C4FA34
+P 7300 6700
+F 0 "#PWR?" H 7300 6650 20  0001 C CNN
+F 1 "+24V" H 7300 6800 30  0000 C CNN
+F 2 "" H 7300 6700 60  0000 C CNN
+F 3 "" H 7300 6700 60  0000 C CNN
+	1    7300 6700
+	0    -1   -1   0
+$EndComp
 $EndSCHEMATC

Commit message: I forget, stuff!
Parts:
- gave numbers to parts that had none: 1
Changed lines of the file:
@@
 $EndComp
 $Comp
-L GND #PWR16
+L GND #PWR20
 U 1 1 54A9BAB0
 P 7750 1500
-F 0 "#PWR16" H 7750 1500 30  0001 C CNN
+F 0 "#PWR20" H 7750 1500 30  0001 C CNN
 F 1 "GND" H 7750 1430 30  0001 C CNN
 F 2 "" H 7750 1500 60  0000 C CNN
@@
 $EndComp
 $Comp
-L +5V #PWR21
+L +5V #PWR25
 U 1 1 54A9D88A
 P 10100 6650
-F 0 "#PWR21" H 10100 6740 20  0001 C CNN
+F 0 "#PWR25" H 10100 6740 20  0001 C CNN
 F 1 "+5V" H 10100 6740 30  0000 C CNN
 F 2 "" H 10100 6650 60  0000 C CNN
@@
 $EndComp
 $Comp
-L GND #PWR20
+L GND #PWR24
 U 1 1 54A9D899
 P 9000 6650
-F 0 "#PWR20" H 9000 6650 30  0001 C CNN
+F 0 "#PWR24" H 9000 6650 30  0001 C CNN
 F 1 "GND" H 9000 6580 30  0001 C CNN
 F 2 "" H 9000 6650 60  0000 C CNN
@@
 $EndComp
 $Comp
-L +24V #PWR25
+L +24V #PWR29
 U 1 1 54BB06EF
 P 10750 800
-F 0 "#PWR25" H 10750 750 20  0001 C CNN
+F 0 "#PWR29" H 10750 750 20  0001 C CNN
 F 1 "+24V" H 10750 900 30  0000 C CNN
 F 2 "" H 10750 800 60  0000 C CNN
@@
 $EndComp
 $Comp
-L GND #PWR19
+L GND #PWR23
 U 1 1 54BB0DB5
 P 8500 800
-F 0 "#PWR19" H 8500 800 30  0001 C CNN
+F 0 "#PWR23" H 8500 800 30  0001 C CNN
 F 1 "GND" H 8500 730 30  0001 C CNN
 F 2 "" H 8500 800 60  0000 C CNN
@@
 $EndComp
 $Comp
-L +5V #PWR22
+L +5V #PWR26
 U 1 1 54BB2061
 P 10400 5450
-F 0 "#PWR22" H 10400 5540 20  0001 C CNN
+F 0 "#PWR26" H 10400 5540 20  0001 C CNN
 F 1 "+5V" H 10400 5540 30  0000 C CNN
 F 2 "" H 10400 5450 60  0000 C CNN
@@
 M-ON/OFF
 $Comp
-L +24V #PWR23
+L +24V #PWR27
 U 1 1 54C20A79
 P 10550 6700
-F 0 "#PWR23" H 10550 6650 20  0001 C CNN
+F 0 "#PWR27" H 10550 6650 20  0001 C CNN
 F 1 "+24V" H 10550 6800 30  0000 C CNN
 F 2 "" H 10550 6700 60  0000 C CNN
@@
 $EndComp
 $Comp
-L GND #PWR24
+L GND #PWR28
 U 1 1 54C20AB0
 P 10550 6900
-F 0 "#PWR24" H 10550 6900 30  0001 C CNN
+F 0 "#PWR28" H 10550 6900 30  0001 C CNN
 F 1 "GND" H 10550 6830 30  0001 C CNN
 F 2 "" H 10550 6900 60  0000 C CNN
@@
 $EndComp
 $Comp
-L GND #PWR18
+L GND #PWR22
 U 1 1 54C261F8
 P 8000 6900
-F 0 "#PWR18" H 8000 6900 30  0001 C CNN
+F 0 "#PWR22" H 8000 6900 30  0001 C CNN
 F 1 "GND" H 8000 6830 30  0001 C CNN
 F 2 "" H 8000 6900 60  0000 C CNN
@@
 $EndComp
 $Comp
-L +5V #PWR17
+L +5V #PWR21
 U 1 1 54C261FE
 P 8000 6700
-F 0 "#PWR17" H 8000 6790 20  0001 C CNN
+F 0 "#PWR21" H 8000 6790 20  0001 C CNN
 F 1 "+5V" H 8000 6790 30  0000 C CNN
 F 2 "" H 8000 6700 60  0000 C CNN
@@
 Connection ~ 1950 1600
 $Comp
-L CONN_4 P?
+L CONN_4 P9
 U 1 1 54C4FA0B
 P 7650 6750
-F 0 "P?" V 7600 6750 50  0000 C CNN
+F 0 "P9" V 7600 6750 50  0000 C CNN
 F 1 "pr28v" V 7700 6750 50  0000 C CNN
 F 2 "" H 7650 6750 60  0000 C CNN
@@
 $EndComp
 $Comp
-L +5V #PWR?
+L +5V #PWR16
 U 1 1 54C4FA18
 P 7300 6600
-F 0 "#PWR?" H 7300 6690 20  0001 C CNN
+F 0 "#PWR16" H 7300 6690 20  0001 C CNN
 F 1 "+5V" H 7300 6690 30  0000 C CNN
 F 2 "" H 7300 6600 60  0000 C CNN
@@
 $EndComp
 $Comp
-L GND #PWR?
+L GND #PWR19
 U 1 1 54C4FA1E
 P 7300 6900
-F 0 "#PWR?" H 7300 6900 30  0001 C CNN
+F 0 "#PWR19" H 7300 6900 30  0001 C CNN
 F 1 "GND" H 7300 6830 30  0001 C CNN
 F 2 "" H 7300 6900 60  0000 C CNN
@@
 $EndComp
 $Comp
-L GND #PWR?
+L GND #PWR18
 U 1 1 54C4FA24
 P 7300 6800
-F 0 "#PWR?" H 7300 6800 30  0001 C CNN
+F 0 "#PWR18" H 7300 6800 30  0001 C CNN
 F 1 "GND" H 7300 6730 30  0001 C CNN
 F 2 "" H 7300 6800 60  0000 C CNN
@@
 $EndComp
 $Comp
-L +24V #PWR?
+L +24V #PWR17
 U 1 1 54C4FA34
 P 7300 6700
-F 0 "#PWR?" H 7300 6650 20  0001 C CNN
+F 0 "#PWR17" H 7300 6650 20  0001 C CNN
 F 1 "+24V" H 7300 6800 30  0000 C CNN
 F 2 "" H 7300 6700 60  0000 C CNN

Commit message: Updated for better 24v section.
Parts:
- removed C6: 0.01uF/50V, ~, symbol CP1
- C1: value 10uf -> 1uf
- R1: value 10K -> 1K
Connections:
- wire segments 263 -> 261
Other:
- moved on the sheet: P2, P7, R2, SHIELD1, SW1
